File: SportModel/SportModel.sch (KiCad schematic (older format))
At the start: 30 parts

Commit message: Added user switch input signal
Parts:
- added J3: UART, Connector_PinHeader_2.54mm:PinHeader_1x04_P2.54mm_Vertical, symbol Connector:Conn_01x04_Male
- added R11: R, Resistor_SMD:R_01005_0402Metric, symbol Device:R
- gave numbers to parts that had none: 27
- renumbered FLASH to FLASH1, RESET to RESET1, USER to USER1
Connections:
- net ED-RESET: now also R11.1; no longer Q2.2 (G), R10.2
- net GND: now also J3.1 (Pin_1)
- net SCL: now also J3.2 (Pin_2)
- net SDA: now also J3.3 (Pin_3)
- net VCC: now also J3.4 (Pin_4)
- net ESP_USER: now reaches U1.5 (GPIO14)
- net ESP_USER: now also C5.1, D3.1 (K), R8.2, USER1.2
- new net: Q2.2 (G), R10.2, R11.2
- no-connect marks 9 -> 8
